File: ov7670.brd (EAGLE design)
At the start: 60.3 x 44.4 mm, 3 parts

Commit message: update
Signed-off-by: Shohei Aoki <shoaok@gmail.com>
Parts:
- moved U$3 0.32 mm to (41.0, 16.8)
Routing:
- net SCL: track 45.0 -> 42.8 mm
- net D1: track 27.5 -> 26.9 mm
Changed lines of the file:
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@@
 <wire x1="60.305" y1="44.4375" x2="0" y2="44.4375" width="0" layer="20"/>
 <wire x1="0" y1="44.4375" x2="0" y2="0" width="0" layer="20"/>
-<dimension x1="17.78" y1="16.8275" x2="40.64" y2="16.8275" x3="29.21" y3="7.9375" textsize="1.778" layer="21"/>
+<dimension x1="17.92" y1="13.0175" x2="40.9575" y2="13.0175" x3="29.43875" y3="8.5725" textsize="1.778" layer="21"/>
 </plain>
 <attributes>
@@
 <element name="U$1" library="ov7670" package="OV7670" value="OV7670" x="27.6225" y="34.925" rot="R90"/>
 <element name="U$2" library="ov7670" package="PMOD_JD" value="PMOD_JD" x="17.92" y="13.0175" rot="MR270"/>
-<element name="U$3" library="ov7670" package="PMOD_JE" value="PMOD_JE" x="40.64" y="16.8275" rot="MR270"/>
+<element name="U$3" library="ov7670" package="PMOD_JE" value="PMOD_JE" x="40.9575" y="16.8275" rot="MR270"/>
 </elements>
 <signals>
@@
 <contactref element="U$2" pad="3"/>
 <contactref element="U$1" pad="SCL"/>
-<wire x1="25.0825" y1="34.925" x2="25.0825" y2="40.005" width="0.762" layer="16"/>
-<wire x1="25.0825" y1="40.005" x2="9.8425" y2="39.6875" width="0.762" layer="16"/>
+<wire x1="25.0825" y1="34.925" x2="25.0825" y2="38.735" width="0.762" layer="16"/>
+<wire x1="25.0825" y1="38.735" x2="9.8425" y2="38.735" width="0.762" layer="16"/>
 <via x="9.8425" y="31.75" extent="1-16" drill="0.8"/>
 <via x="16.51" y="20.32" extent="1-16" drill="0.8"/>
-<wire x1="9.8425" y1="39.6875" x2="9.8425" y2="31.75" width="0.762" layer="16"/>
+<wire x1="9.8425" y1="38.735" x2="9.8425" y2="31.75" width="0.762" layer="16"/>
 <wire x1="9.8425" y1="31.75" x2="16.51" y2="20.32" width="0.762" layer="1"/>
 <wire x1="16.51" y1="20.32" x2="16.65" y2="20.18" width="0.762" layer="16"/>
@@
 <contactref element="U$3" pad="1"/>
 <contactref element="U$1" pad="D7"/>
-<wire x1="31.75" y1="16.8275" x2="34.29" y2="16.8275" width="0.762" layer="16"/>
+<wire x1="31.75" y1="16.8275" x2="34.6075" y2="16.8275" width="0.762" layer="16"/>
 <wire x1="31.75" y1="4.445" x2="31.75" y2="16.8275" width="0.762" layer="16"/>
 <wire x1="48.895" y1="4.445" x2="31.75" y2="4.445" width="0.762" layer="16"/>
@@
 <contactref element="U$3" pad="2"/>
 <contactref element="U$1" pad="D5"/>
-<wire x1="35.56" y1="18.7325" x2="35.56" y2="32.0675" width="0.762" layer="16"/>
-<wire x1="36.83" y1="17.4625" x2="35.56" y2="18.7325" width="0.762" layer="16"/>
-<wire x1="36.83" y1="16.8275" x2="36.83" y2="17.4625" width="0.762" layer="16"/>
-<wire x1="35.56" y1="32.0675" x2="35.2425" y2="32.385" width="0.762" layer="16"/>
+<wire x1="37.1475" y1="20.32" x2="35.2425" y2="21.59" width="0.762" layer="16"/>
+<wire x1="35.2425" y1="21.59" x2="35.2425" y2="32.385" width="0.762" layer="16"/>
+<wire x1="37.1475" y1="16.8275" x2="37.1475" y2="20.32" width="0.762" layer="16"/>
 </signal>
 <signal name="D3">
 <contactref element="U$3" pad="3"/>
 <contactref element="U$1" pad="D3"/>
-<wire x1="39.37" y1="16.8275" x2="39.37" y2="20.32" width="0.762" layer="16"/>
-<via x="39.37" y="20.32" extent="1-16" drill="0.8"/>
-<wire x1="39.37" y1="20.32" x2="32.385" y2="20.32" width="0.762" layer="1"/>
-<via x="32.385" y="20.32" extent="1-16" drill="0.8"/>
-<wire x1="32.385" y1="20.32" x2="32.7025" y2="32.385" width="0.762" layer="16"/>
+<wire x1="39.6875" y1="16.8275" x2="39.6875" y2="20.32" width="0.762" layer="16"/>
+<via x="39.6875" y="20.32" extent="1-16" drill="0.8"/>
+<wire x1="39.6875" y1="20.32" x2="32.7025" y2="20.32" width="0.762" layer="1"/>
+<via x="32.7025" y="20.32" extent="1-16" drill="0.8"/>
+<wire x1="32.7025" y1="20.32" x2="32.7025" y2="32.385" width="0.762" layer="16"/>
 </signal>
 <signal name="D1">
 <contactref element="U$3" pad="4"/>
 <contactref element="U$1" pad="D1"/>
-<wire x1="41.91" y1="16.8275" x2="42.2275" y2="17.145" width="0.762" layer="16"/>
-<wire x1="42.2275" y1="17.145" x2="42.2275" y2="21.2725" width="0.762" layer="16"/>
+<wire x1="42.2275" y1="16.8275" x2="42.2275" y2="21.2725" width="0.762" layer="16"/>
 <wire x1="42.2275" y1="21.2725" x2="40.9575" y2="22.5425" width="0.762" layer="16"/>
 <wire x1="40.9575" y1="22.5425" x2="38.1" y2="22.5425" width="0.762" layer="16"/>
 <via x="38.1" y="22.5425" extent="1-16" drill="0.8"/>
-<wire x1="38.1" y1="22.5425" x2="29.845" y2="22.5425" width="0.762" layer="1"/>
-<via x="29.845" y="22.5425" extent="1-16" drill="0.8"/>
-<wire x1="29.845" y1="22.5425" x2="30.1625" y2="22.86" width="0.762" layer="16"/>
-<wire x1="30.1625" y1="22.86" x2="30.1625" y2="32.385" width="0.762" layer="16"/>
+<wire x1="38.1" y1="22.5425" x2="30.1625" y2="22.5425" width="0.762" layer="1"/>
+<via x="30.1625" y="22.5425" extent="1-16" drill="0.8"/>
+<wire x1="30.1625" y1="22.5425" x2="30.1625" y2="32.385" width="0.762" layer="16"/>
 </signal>
 <signal name="D6">
 <contactref element="U$3" pad="7"/>
 <contactref element="U$1" pad="D6"/>
-<via x="34.29" y="6.0325" extent="1-16" drill="0.8"/>
-<wire x1="34.29" y1="6.0325" x2="51.7525" y2="6.0325" width="0.762" layer="1"/>
+<via x="34.6075" y="6.0325" extent="1-16" drill="0.8"/>
+<wire x1="34.6075" y1="6.0325" x2="51.7525" y2="6.0325" width="0.762" layer="1"/>
 <via x="51.7525" y="6.0325" extent="1-16" drill="0.8"/>
 <wire x1="51.7525" y1="6.0325" x2="51.7525" y2="12.30803125" width="0.762" layer="16"/>
 <wire x1="51.7525" y1="12.30803125" x2="51.80526875" y2="12.756565625" width="0.762" layer="16"/>
 <wire x1="51.80526875" y1="12.756565625" x2="51.7525" y2="12.82340625" width="0.762" layer="16"/>
-<wire x1="34.29" y1="14.2875" x2="34.29" y2="6.0325" width="0.762" layer="16"/>
+<wire x1="34.6075" y1="14.2875" x2="34.6075" y2="6.0325" width="0.762" layer="16"/>
 <wire x1="51.435" y1="24.13" x2="39.0525" y2="36.5125" width="0.762" layer="16"/>
 <wire x1="39.0525" y1="36.5125" x2="38.9602375" y2="36.5125" width="0.762" layer="16"/>
@@
 <contactref element="U$3" pad="8"/>
 <contactref element="U$1" pad="D4"/>
-<wire x1="36.83" y1="14.2875" x2="36.83" y2="7.62" width="0.762" layer="16"/>
-<via x="36.83" y="7.62" extent="1-16" drill="0.8"/>
+<wire x1="37.1475" y1="14.2875" x2="37.1475" y2="7.62" width="0.762" layer="16"/>
+<via x="37.1475" y="7.62" extent="1-16" drill="0.8"/>
 <via x="53.34" y="7.62" extent="1-16" drill="0.8"/>
 <wire x1="53.34" y1="7.62" x2="53.34" y2="25.0825" width="0.762" layer="16"/>
@@
 <wire x1="36.07870625" y1="38.4175" x2="32.7025" y2="38.4175" width="0.762" layer="16"/>
 <wire x1="32.7025" y1="38.4175" x2="32.7025" y2="34.925" width="0.762" layer="16"/>
-<wire x1="36.83" y1="7.62" x2="53.34" y2="7.62" width="0.762" layer="1"/>
+<wire x1="37.1475" y1="7.62" x2="53.34" y2="7.62" width="0.762" layer="1"/>
 </signal>
 <signal name="D2">
 <contactref element="U$3" pad="9"/>
 <contactref element="U$1" pad="D2"/>
-<wire x1="39.37" y1="14.2875" x2="39.37" y2="9.2075" width="0.762" layer="16"/>
-<via x="39.37" y="9.2075" extent="1-16" drill="0.8"/>
+<wire x1="39.6875" y1="14.2875" x2="39.6875" y2="9.2075" width="0.762" layer="16"/>
+<via x="39.6875" y="9.2075" extent="1-16" drill="0.8"/>
 <wire x1="30.1625" y1="34.925" x2="30.1625" y2="40.005" width="0.762" layer="16"/>
 <wire x1="35.23515" y1="40.005" x2="35.60815" y2="40.0605" width="0.762" layer="16"/>
@@
 <wire x1="35.60815" y1="40.0605" x2="41.8545" y2="40.0605" width="0.762" layer="16"/>
 <via x="55.245" y="9.2075" extent="1-16" drill="0.8"/>
-<wire x1="55.245" y1="9.2075" x2="39.37" y2="9.2075" width="0.762" layer="1"/>
+<wire x1="55.245" y1="9.2075" x2="39.6875" y2="9.2075" width="0.762" layer="1"/>
 <wire x1="41.8545" y1="40.0605" x2="54.9275" y2="26.035" width="0.762" layer="16"/>
 <wire x1="54.9275" y1="26.035" x2="55.245" y2="9.2075" width="0.762" layer="16"/>
@@
 <contactref element="U$3" pad="10"/>
 <contactref element="U$1" pad="D0"/>
-<via x="41.91" y="10.7922" extent="1-16" drill="0.8"/>
-<wire x1="41.91" y1="10.7922" x2="41.9072" y2="10.795" width="0.762" layer="1"/>
-<wire x1="41.91" y1="14.2875" x2="41.91" y2="10.7922" width="0.762" layer="16"/>
+<via x="42.2275" y="10.7922" extent="1-16" drill="0.8"/>
+<wire x1="42.2275" y1="10.7922" x2="41.9072" y2="10.795" width="0.762" layer="1"/>
+<wire x1="42.2275" y1="14.2875" x2="42.2275" y2="10.7922" width="0.762" layer="16"/>
 <via x="57.15" y="10.795" extent="1-16" drill="0.8"/>
 <wire x1="57.15" y1="10.795" x2="57.15" y2="26.9875" width="0.762" layer="16"/>

Commit message: temporal commit
Parts:
- removed U$1: OV7670, ov7670:OV7670
- added D6: OV7670, ov7670:OV7670
- moved U$2 5.09 mm to (23.0, 12.7), flipped to the top, turned to 0 degrees
- moved U$3 2.86 mm to (41.0, 14.0), flipped to the top, turned to 0 degrees
Connections:
- removed net D6: U$1.D6, U$3.7
- removed net GND: U$1.GND, U$2.5
- removed net PLCK: U$1.PLCK, U$2.9
- new net N$1: D6.GND, U$3.P$6
- new net N$6: D6.D6, U$2.7
- new net PCLK: D6.PCLK, U$3.P$9
- net 3V3: now also D6.3V3; no longer U$1.3V3
- net D0: now also D6.D0, U$2.10; no longer U$1.D0, U$3.10
- net D1: now also D6.D1, U$2.4; no longer U$1.D1, U$3.4
- net D2: now also D6.D2, U$2.9; no longer U$1.D2, U$3.9
- net D3: now also D6.D3, U$2.3; no longer U$1.D3, U$3.3
- net D4: now also D6.D4, U$2.8; no longer U$1.D4, U$3.8
- net D5: now also D6.D5, U$2.2; no longer U$1.D5, U$3.2
- net D7: now also D6.D7, U$2.1; no longer U$1.D7, U$3.1
- net HREF: now also D6.HREF, U$3.P$10; no longer U$1.HREF, U$2.10
- net SCL: now also D6.SCL, U$3.P$3; no longer U$1.SCL, U$2.3
- net SDA: now also D6.SDA, U$3.P$7; no longer U$1.SDA, U$2.7
- net VSYNC: now also D6.VSYNC, U$3.P$4; no longer U$1.VSYNC, U$2.4
- net XCLK: now also D6.XCLK, U$3.P$8; no longer U$1.XCLK, U$2.8
Routing:
- net GND: track 84.6 -> 0.00 mm
- net PCLK: track 0.00 -> 80.9 mm, vias 0 -> 2
- net N$6: track 0.00 -> 67.8 mm, vias 0 -> 2
- net D6: track 66.5 -> 0.00 mm, vias 2 -> 0
- net SCL: track 42.8 -> 106.6 mm
- net D1: track 26.9 -> 87.9 mm, vias 2 -> 0
- net PLCK: track 59.7 -> 0.00 mm, vias 2 -> 0
- net 3V3: track 74.5 -> 17.5 mm
- net N$1: track 0.00 -> 31.2 mm, vias 0 -> 2
- net SDA: track 40.2 -> 70.5 mm, vias 2 -> 0
- net D7: track 64.9 -> 41.0 mm, vias 0 -> 2
- net XCLK: track 44.6 -> 65.4 mm, vias 2 -> 0
- net D5: track 16.6 -> 36.0 mm, vias 0 -> 2
- net VSYNC: track 17.5 -> 34.6 mm
- net D3: track 22.5 -> 30.9 mm
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- removed copper zone on layer 16, net GND
Other:
- board size 60.3 x 44.4 mm -> 66.3 x 53.3 mm

Commit message: update
Parts:
- moved D6 8.82 mm to (35.2, 27.0)
- moved U$2 8.82 mm to (30.6, 8.26)
- moved U$3 8.82 mm to (48.6, 9.53)
Connections:
- net N$1 renamed GND
Routing:
- net D1: track 87.9 -> 95.5 mm
- net HREF: track 72.2 -> 76.8 mm
- net PCLK: track 80.9 -> 85.4 mm
- net D0: track 76.6 -> 80.7 mm
- net N$6: track 67.8 -> 71.9 mm
- net D2: track 74.2 -> 78.0 mm
- net D4: track 71.4 -> 75.1 mm
- net SCL: track 106.6 -> 108.7 mm
- net SDA: track 70.5 -> 71.4 mm
- net XCLK: track 65.4 -> 66.4 mm
- net 3V3: track 17.5 -> 18.3 mm
- added copper zone on layer 16, net GND
Other:
- board size 66.3 x 53.3 mm -> 54.3 x 46.7 mm

Commit message: update
Connections:
- net GND: now also U$3.P$5; no longer U$3.P$6
Routing:
- net GND: track 31.2 -> 30.7 mm
Changed lines of the file:
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@@
 </polygon>
 <contactref element="D6" pad="GND"/>
-<contactref element="U$3" pad="P$6"/>
 <wire x1="45.4025" y1="29.5275" x2="45.4025" y2="33.9725" width="0.762" layer="16"/>
 <via x="45.4025" y="33.9725" extent="1-16" drill="0.8"/>
 <wire x1="45.4025" y1="33.9725" x2="49.53" y2="33.9725" width="0.762" layer="1"/>
-<wire x1="49.53" y1="33.9725" x2="54.9275" y2="14.9225" width="0.762" layer="1"/>
-<via x="54.9275" y="14.9225" extent="1-16" drill="0.8"/>
-<wire x1="54.9275" y1="12.065" x2="54.9275" y2="14.9225" width="0.762" layer="16"/>
+<wire x1="49.53" y1="33.9725" x2="52.3875" y2="14.9225" width="0.762" layer="1"/>
+<via x="52.3875" y="14.9225" extent="1-16" drill="0.8"/>
 <polygon width="0.762" layer="16">
 <vertex x="6.35" y="0"/>
@@
 <vertex x="60.0075" y="0.635"/>
 </polygon>
+<contactref element="U$3" pad="P$5"/>
+<wire x1="52.3875" y1="14.9225" x2="52.3875" y2="12.065" width="0.762" layer="16"/>
 </signal>
 </signals>
